File: matrix.kicad_sch (KiCad schematic)
At the start: 120 parts, among them SW10 #8, SW11 #9, SW12 #0, SW13 -_, SW14 =+, SW15 \|, SW16 `~, SW17 Tab, SW18 Q, SW19 W, SW2 Esc, SW20 E, SW21 R, SW22 T, SW23 Y, SW24 U, SW25 I, SW26 O, SW27 P, SW28 [{, SW29 ]}, SW3 #1, SW30 Bksp, SW31 Ctrl, SW32 A, SW33 S, SW34 D, SW35 F, SW36 G, SW37 H, SW38 J, SW39 K, SW4 #2, SW40 L, SW41 ;:, SW42 '", SW43 Enter, SW44 Shift, SW45 Z, SW46 X, SW47 C, SW48 V, SW49 B, SW5 #3, SW50 N, SW51 M, SW52 ,<, SW53 .>, SW54 /?, SW55 Shift, SW56 Fn, SW57 Win, SW58 Alt, SW59 Space, SW6 #4, SW60 Alt, SW61 Ctrl, SW7 #5, SW8 #6, SW9 #7

Commit message: Fixed lonely column.
Connections:
- net col13: no longer SW56.2
- net col14: now also SW56.2
Other:
- moved on the sheet: D55, SW56
Changed lines of the file:
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@@
 	)
 	(junction
+		(at 255.27 114.3)
+		(diameter 0)
+		(color 0 0 0 0)
+	)
+	(junction
 		(at 209.55 66.04)
 		(diameter 0)
@@
 	)
 	(junction
-		(at 229.87 121.92)
+		(at 77.47 49.53)
 		(diameter 0)
 		(color 0 0 0 0)
 	)
 	(junction
-		(at 77.47 49.53)
+		(at 168.91 49.53)
 		(diameter 0)
 		(color 0 0 0 0)
 	)
 	(junction
-		(at 168.91 49.53)
+		(at 62.23 121.92)
 		(diameter 0)
 		(color 0 0 0 0)
 	)
 	(junction
-		(at 62.23 121.92)
+		(at 245.11 121.92)
 		(diameter 0)
 		(color 0 0 0 0)
@@
 	)
 	(junction
-		(at 240.03 114.3)
-		(diameter 0)
-		(color 0 0 0 0)
-	)
-	(junction
 		(at 163.83 90.17)
 		(diameter 0)
@@
 	(wire
 		(pts
+			(xy 255.27 41.91) (xy 255.27 114.3)
+		)
+		(stroke
+			(width 0)
+			(type default)
+		)
+	)
+	(wire
+		(pts
 			(xy 199.39 49.53) (xy 214.63 49.53)
 		)
@@
 	(wire
 		(pts
+			(xy 245.11 121.92) (xy 260.35 121.92)
+		)
+		(stroke
+			(width 0)
+			(type default)
+		)
+	)
+	(wire
+		(pts
 			(xy 107.95 121.92) (xy 123.19 121.92)
 		)
@@
 	(wire
 		(pts
+			(xy 255.27 114.3) (xy 255.27 149.86)
+		)
+		(stroke
+			(width 0)
+			(type default)
+		)
+	)
+	(wire
+		(pts
 			(xy 107.95 73.66) (xy 123.19 73.66)
 		)
@@
 	(wire
 		(pts
-			(xy 229.87 121.92) (xy 260.35 121.92)
-		)
-		(stroke
-			(width 0)
-			(type default)
-		)
-	)
-	(wire
-		(pts
 			(xy 123.19 121.92) (xy 138.43 121.92)
 		)
@@
 	(wire
 		(pts
-			(xy 255.27 41.91) (xy 255.27 149.86)
-		)
-		(stroke
-			(width 0)
-			(type default)
-		)
-	)
-	(wire
-		(pts
 			(xy 118.11 90.17) (xy 118.11 114.3)
 		)
@@
 	(wire
 		(pts
-			(xy 240.03 114.3) (xy 240.03 149.86)
+			(xy 240.03 90.17) (xy 240.03 149.86)
 		)
 		(stroke
@@
 	(wire
 		(pts
-			(xy 214.63 121.92) (xy 229.87 121.92)
+			(xy 214.63 121.92) (xy 245.11 121.92)
 		)
 		(stroke
@@
 	(wire
 		(pts
-			(xy 240.03 90.17) (xy 240.03 114.3)
-		)
-		(stroke
-			(width 0)
-			(type default)
-		)
-	)
-	(wire
-		(pts
 			(xy 118.11 66.04) (xy 118.11 90.17)
 		)
@@
 	(symbol
 		(lib_id "Switch:SW_Push")
-		(at 234.95 114.3 0)
+		(at 250.19 114.3 0)
 		(unit 1)
 		(exclude_from_sim no)
@@
 		(fields_autoplaced yes)
 		(property "Reference" "SW56"
-			(at 234.95 106.68 0)
+			(at 250.19 106.68 0)
 			(effects
 				(font
@@
 		)
 		(property "Value" "Fn"
-			(at 234.95 109.22 0)
+			(at 250.19 109.22 0)
 			(effects
 				(font
@@
 		)
 		(property "Footprint" "PCM_marbastlib-xp-choc:SW_choc_v2_HS_CPG135001S30_1u"
-			(at 234.95 109.22 0)
+			(at 250.19 109.22 0)
 			(effects
 				(font
@@
 		)
 		(property "Datasheet" "~"
-			(at 234.95 109.22 0)
+			(at 250.19 109.22 0)
 			(effects
 				(font
@@
 		)
 		(property "Description" "Push button switch, generic, two pins"
-			(at 234.95 114.3 0)
+			(at 250.19 114.3 0)
 			(effects
 				(font
@@
 	(symbol
 		(lib_id "Device:D")
-		(at 229.87 118.11 90)
+		(at 245.11 118.11 90)
 		(unit 1)
 		(exclude_from_sim no)
@@
 		(on_board yes)
 		(dnp no)
-		(fields_autoplaced yes)
 		(property "Reference" "D55"
-			(at 232.41 116.8399 90)
+			(at 247.65 116.8399 90)
 			(effects
 				(font
@@
 		)
 		(property "Value" "D"
-			(at 232.41 119.3799 90)
+			(at 247.65 119.3799 90)
 			(effects
 				(font
@@
 		)
 		(property "Footprint" "Diode_SMD:D_0805_2012Metric"
-			(at 229.87 118.11 0)
+			(at 245.11 118.11 0)
 			(effects
 				(font
@@
 		)
 		(property "Datasheet" "~"
-			(at 229.87 118.11 0)
+			(at 245.11 118.11 0)
 			(effects
 				(font
@@
 		)
 		(property "Description" "Diode"
-			(at 229.87 118.11 0)
+			(at 245.11 118.11 0)
 			(effects
 				(font
@@
 		)
 		(property "Sim.Device" "D"
-			(at 229.87 118.11 0)
+			(at 245.11 118.11 0)
 			(effects
 				(font
@@
 		)
 		(property "Sim.Pins" "1=K 2=A"
-			(at 229.87 118.11 0)
+			(at 245.11 118.11 0)
 			(effects
 				(font

Commit message: Change footprints, fix errors, WIP BOM.
Parts:
- D1, D10, D11, D12, D13, D14, D15, D16, D17, D18, D19, D2, D20, D21, D22, D23, D24, D25, D26, D27, D28, D29, D3, D30, D31, D32, D33, D34, D35, D36, D37, D38, D39, D4, D40, D41, D42, D43, D44, D45, D46, D47, D48, D49, D5, D50, D51, D52, D53, D54, D55, D56, D57, D58, D59, D6, D60, D7, D8, D9: footprint Diode_SMD:D_0805_2012Metric -> Diode_SMD:D_SOD-323; JLCPCB Part (none) -> C2128
- SW13: value -_ -> Minus
- SW14: value =+ -> Equals
- SW15: value \| -> Backslash
- SW16: value `~ -> Grave
- SW41: value ;: -> Semi
- SW42: value '" -> Quote
- SW52: value ,< -> Comma
- SW53: value .> -> Dot
- SW54: value /? -> Slash
