File: kicad/keyboard.kicad_pcb (KiCad board)
At the start: 2 copper layers, 293.7 x 209.5 mm, 161 parts, among them J2 Conn_01x06, SW2 SW_Push, U5 RP2040, U6 PRTR5V0U2X, U7 NCP1117-3.3_SOT223, U8 W25Q128JVS, Y2 Crystal_GND24_Small

Commit message: Complete routing and fill zones.
Parts:
- moved U8 2.66 mm to (8.89, 88.9)
Connections:
- R10 pad 2: GND -> Net-(R10-Pad2)
- R9 pad 2: GND -> Net-(R10-Pad2)
- USB2 pad 1: GND -> Net-(R10-Pad2)
- USB2 pad 12: GND -> Net-(R10-Pad2)
- USB2 pad 13: GND -> Earth
Routing:
- net GND: track 242.3 -> 274.2 mm, vias 19 -> 27
- net +3V3: track 156.8 -> 169.4 mm, vias 10 -> 12
- net /RUN: track 20.0 -> 30.4 mm, vias 1 -> 0
- net /CS: track 60.2 -> 54.9 mm
- net +1V1: track 19.8 -> 23.9 mm
- net (no net): track 0.00 -> 3.67 mm, vias 0 -> 4
- net /SD0: track 15.8 -> 12.4 mm
- net /SD3: track 21.0 -> 18.1 mm
- net /SCLK: track 18.9 -> 16.0 mm
- net /SD2: track 8.41 -> 6.44 mm
- net /SD1: track 8.77 -> 7.34 mm
- net Earth: vias 0 -> 5
- added copper zone on F.Cu, net +1V1
- added copper zone on B.Cu, net Earth
- added copper zone on F.Cu, net Earth
- added copper zone on B.Cu, net GND
- added copper zone on F.Cu, net GND

Commit message: Update.
Connections:
- R10 pad 2: Net-(R10-Pad2) -> GND
- R9 pad 2: Net-(R10-Pad2) -> GND
- USB2 pad 1: Net-(R10-Pad2) -> GND
- USB2 pad 12: Net-(R10-Pad2) -> GND
Other:
- board size 293.7 x 209.5 mm -> 287.3 x 98.4 mm
Changed lines of the file:
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@@
 	(net 119 "unconnected-(U5-GPIO9-Pad12)")
 	(net 120 "unconnected-(U5-GPIO10-Pad13)")
-	(net 121 "Net-(R10-Pad2)")
 	(footprint "Diode_SMD:D_SOD-323"
 		(layer "F.Cu")
@@
 			(layers "F.Cu" "F.Paste" "F.Mask")
 			(roundrect_rratio 0.25)
-			(net 121 "Net-(R10-Pad2)")
+			(net 84 "GND")
 			(pintype "passive")
 		)
@@
 			(size 0.6 2.45)
 			(layers "F.Cu" "F.Paste" "F.Mask")
-			(net 121 "Net-(R10-Pad2)")
+			(net 84 "GND")
 			(pinfunction "GND")
 			(pintype "input")
@@
 			(size 0.6 2.45)
 			(layers "F.Cu" "F.Paste" "F.Mask")
-			(net 121 "Net-(R10-Pad2)")
+			(net 84 "GND")
 			(pinfunction "GND")
 			(pintype "input")
@@
 			(layers "F.Cu" "F.Paste" "F.Mask")
 			(roundrect_rratio 0.25)
-			(net 121 "Net-(R10-Pad2)")
+			(net 84 "GND")
 			(pintype "passive")
 		)
@@
 		(tags "Kailh Choc Keyswitch Switch CPG1350 V1 CPG1353 V2 Hotswap Cutout")
 		(property "Reference" "K_14"
-			(at 0 9 0)
+			(at 0 9 180)
 			(layer "B.SilkS")
 			(effects
@@
 		)
 		(property "Value" "KEYSW"
-			(at 0 -9 0)
+			(at 0 -9 180)
 			(layer "B.Fab")
 			(effects
@@
 		)
 		(property "Footprint" "PCM_Switch_Keyboard_Hotswap_Kailh:SW_Hotswap_Kailh_Choc_V1V2"
-			(at 0 0 0)
+			(at 0 0 180)
 			(layer "B.Fab")
 			(hide yes)
@@
 		)
 		(property "Datasheet" ""
-			(at 0 0 0)
+			(at 0 0 180)
 			(layer "B.Fab")
 			(hide yes)
@@
 		)
 		(property "Description" ""
-			(at 0 0 0)
+			(at 0 0 180)
 			(layer "B.Fab")
 			(hide yes)
@@
 			(layer "F.Fab")
 		)
+		(fp_text user "18x17 spacing"
+			(at 0 7.6 180)
+			(layer "Dwgs.User")
+			(effects
+				(font
+					(size 1 1)
+					(thickness 0.15)
+				)
+			)
+		)
+		(fp_text user "LED"
+			(at 0 4.7625 180)
+			(unlocked yes)
+			(layer "Cmts.User")
+			(effects
+				(font
+					(size 1 1)
+					(thickness 0.15)
+				)
+			)
+		)
+		(fp_text user "19.05 spacing"
+			(at 0 8.7 180)
+			(layer "Eco1.User")
+			(effects
+				(font
+					(size 1 1)
+					(thickness 0.15)
+				)
+			)
+		)
 		(fp_text user "${REFERENCE}"
-			(at 0 0 0)
+			(at 0 0 180)
 			(layer "B.Fab")
 			(effects
@@
 		(layer "Edge.Cuts")
 	)
-	(gr_arc
-		(start 285.75 101.6)
-		(mid 288.556298 102.762438)
-		(end 289.71875 105.56875)
-		(stroke
-			(width 0.2)
-			(type default)
-		)
-		(layer "Edge.Cuts")
-	)
-	(gr_line
-		(start 0 204.7875)
-		(end 285.75 204.7875)
-		(stroke
-			(width 0.2)
-			(type solid)
-		)
-		(layer "Edge.Cuts")
-	)
 	(gr_line
-		(start -0.79375 5.55625)
+		(start -0.79375 5.36575)
 		(end -0.79375 89.69375)
 		(stroke
@@
 	)
 	(gr_line
-		(start 282.575 1.5875)
-		(end 24.60625 1.5875)
+		(start 282.575 1.397)
+		(end 24.60625 1.397)
 		(stroke
 			(width 0.2)
@@
 	)
 	(gr_line
-		(start 285.75 101.6)
-		(end 0 101.6)
-		(stroke
-			(width 0.2)
-			(type solid)
-		)
-		(layer "Edge.Cuts")
-	)
-	(gr_line
-		(start 12.7 1.5875)
-		(end 3.175 1.5875)
+		(start 12.7 1.397)
+		(end 3.175 1.397)
 		(stroke
 			(width 0.2)
@@
 	)
 	(gr_arc
-		(start 289.71875 200.81875)
-		(mid 288.556333 203.625098)
-		(end 285.75 204.7875)
-		(stroke
-			(width 0.2)
-			(type default)
-		)
-		(layer "Edge.Cuts")
-	)
-	(gr_arc
-		(start 24.60625 1.5875)
-		(mid 24.044984 1.355016)
-		(end 23.8125 0.79375)
+		(start 24.60625 1.397)
+		(mid 24.044999 1.164501)
+		(end 23.8125 0.60325)
 		(stroke
 			(width 0.2)
@@
 	(gr_line
 		(start 286.54375 89.69375)
-		(end 286.54375 5.55625)
+		(end 286.54375 5.36575)
 		(stroke
 			(width 0.2)
@@
 	)
 	(gr_arc
-		(start 13.49375 0.79375)
-		(mid 13.261266 1.355016)
-		(end 12.7 1.5875)
+		(start 13.49375 0.60325)
+		(mid 13.261266 1.164516)
+		(end 12.7 1.397)
 		(stroke
 			(width 0.2)
@@
 	)
 	(gr_arc
-		(start 282.575 1.5875)
-		(mid 285.38133 2.74992)
-		(end 286.54375 5.55625)
+		(start 282.575 1.397)
+		(mid 285.381348 2.559417)
+		(end 286.54375 5.36575)
 		(stroke
 			(width 0.2)
@@
 		(layer "Edge.Cuts")
 	)
-	(gr_line
-		(start -3.96875 105.56875)
-		(end -3.96875 200.81875)
-		(stroke
-			(width 0.2)
-			(type solid)
-		)
-		(layer "Edge.Cuts")
-	)
 	(gr_arc
-		(start -0.79375 5.55625)
-		(mid 0.36867 2.74992)
-		(end 3.175 1.5875)
+		(start -0.79375 5.36575)
+		(mid 0.36867 2.55942)
+		(end 3.175 1.397)
 		(stroke
 			(width 0.2)
@@
 	(gr_line
 		(start 13.49375 -4.7625)
-		(end 13.49375 0.79375)
+		(end 13.49375 0.60325)
 		(stroke
 			(width 0.2)
@@
 	(gr_line
 		(start 23.8125 -4.7625)
-		(end 23.8125 0.79375)
-		(stroke
-			(width 0.2)
-			(type default)
-		)
-		(layer "Edge.Cuts")
-	)
-	(gr_line
-		(start 289.71875 200.81875)
-		(end 289.71875 105.56875)
-		(stroke
-			(width 0.2)
-			(type solid)
-		)
-		(layer "Edge.Cuts")
-	)
-	(gr_arc
-		(start -3.96875 105.56875)
-		(mid -2.80633 102.76242)
-		(end 0 101.6)
+		(end 23.8125 0.60325)
 		(stroke
 			(width 0.2)
@@
 		(layer "Edge.Cuts")
 	)
-	(gr_arc
-		(start 0 204.7875)
-		(mid -2.80633 203.62508)
-		(end -3.96875 200.81875)
-		(stroke
-			(width 0.2)
-			(type default)
-		)
-		(layer "Edge.Cuts")
-	)
 	(segment
 		(start 7.391063 79.095937)
@@
 	)
 	(segment
+		(start 17.526 81.33589)
+		(end 17.526 81.788)
+		(width 0.2)
+		(layer "F.Cu")
+		(net 86)
+	)
+	(segment
 		(start 28.121686 81.715685)
 		(end 29.573371 80.264)
@@
 	)
 	(segment
-		(start 17.526 81.33589)
-		(end 17.526 81.534)
-		(width 0.2)
-		(layer "F.Cu")
-		(net 86)
-	)
-	(segment
 		(start 9.7452 82.75)
 		(end 9.4944 82.4992)
@@
 		(polygon
 			(pts
-				(xy 16.891 79.502) (xy 22.86 79.502) (xy 22.86 85.598) (xy 16.891 85.598)
+				(xy 22.86 85.598) (xy 16.891 85.598) (xy 16.891 79.502) (xy 22.86 79.502)
+			)
+		)
+		(polygon
+			(pts
+				(xy 20.955 80.645) (xy 20.955 80.645) (xy 18.034 80.645) (xy 18.034 84.455) (xy 21.717 84.455) (xy 21.717 80.645)
 			)
 		)
@@
 		(polygon
 			(pts
-				(xy 290.322 -7.874) (xy 291.465 99.822) (xy -9.017 97.409) (xy -8.255 -8.636)
+				(xy 290.449 -7.874) (xy 291.592 99.822) (xy -8.89 97.409) (xy -8.128 -8.636)
+			)
+		)
+		(polygon
+			(pts
+				(xy 26.924 88.9) (xy 36.576 89.027) (xy 36.703 80.518) (xy 32.385 80.518) (xy 27.178 80.518)
 			)
 		)
 		(polygon
 			(pts
-				(xy 26.797 88.9) (xy 36.449 89.027) (xy 36.576 80.518) (xy 32.258 80.518) (xy 27.051 80.518)
+				(xy 16.891 79.502) (xy 17.018 79.502) (xy 16.891 79.502) (xy 16.891 85.598) (xy 22.86 85.598) (xy 22.86 79.502)
 			)
 		)
 		(polygon
 			(pts
-				(xy 12.7 -5.334) (xy 12.7 4.064) (xy 26.67 4.064) (xy 26.67 -5.334)
+				(xy 12.827 4.064) (xy 26.797 4.064) (xy 26.797 -5.334) (xy 12.827 -5.334)
 			)
 		)
@@
 		(polygon
 			(pts
-				(xy 27.305 80.899) (xy 35.941 80.899) (xy 36.068 88.773) (xy 27.305 88.519) (xy 27.305 80.899)
+				(xy 27.305 80.899) (xy 35.941 80.899) (xy 36.068 88.773) (xy 27.305 88.519)
 			)
 		)
