File: kicad/keyboard.kicad_sch (KiCad schematic)
At the start: 157 parts, among them J2 Conn_01x06, SW2 SW_Push, U5 RP2040, U6 PRTR5V0U2X, U7 NCP1117-3.3_SOT223, U8 W25Q128JVS, Y2 Crystal_GND24_Small

Commit message: Complete routing and fill zones.
Connections:
- net Earth: now also USB2.13 (SHIELD)
- net GND: no longer R10.2, R9.2, USB2.1 (GND), USB2.12 (GND), USB2.13 (SHIELD)
- new net: R10.2, R9.2, USB2.1 (GND), USB2.12 (GND)
Changed lines of the file:
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@@
 	)
 	(junction
+		(at 127 190.5)
+		(diameter 0)
+		(color 0 0 0 0)
+	)
+	(junction
 		(at 147.32 210.82)
 		(diameter 0)
@@
 	)
 	(junction
-		(at 137.16 193.04)
-		(diameter 0)
-		(color 0 0 0 0)
-	)
-	(junction
 		(at 68.58 162.56)
 		(diameter 0)
@@
 	)
 	(junction
-		(at 127 193.04)
-		(diameter 0)
-		(color 0 0 0 0)
-	)
-	(junction
 		(at 274.32 24.13)
 		(diameter 0)
@@
 	)
 	(junction
-		(at 127 190.5)
-		(diameter 0)
-		(color 0 0 0 0)
-	)
-	(junction
 		(at 132.08 165.1)
 		(diameter 0)
@@
 	)
 	(junction
+		(at 137.16 193.04)
+		(diameter 0)
+		(color 0 0 0 0)
+	)
+	(junction
 		(at 364.49 35.56)
 		(diameter 0)
@@
 	(wire
 		(pts
-			(xy 127 193.04) (xy 127 195.58)
-		)
-		(stroke
-			(width 0)
-			(type default)
-		)
-	)
-	(wire
-		(pts
 			(xy 137.16 193.04) (xy 146.05 193.04)
 		)
@@
 	(wire
 		(pts
-			(xy 127 193.04) (xy 137.16 193.04)
-		)
-		(stroke
-			(width 0)
-			(type default)
-		)
-	)
-	(wire
-		(pts
 			(xy 246.38 269.24) (xy 252.73 269.24)
 		)
@@
 	(wire
 		(pts
+			(xy 127 193.04) (xy 137.16 193.04)
+		)
+		(stroke
+			(width 0)
+			(type default)
+		)
+	)
+	(wire
+		(pts
 			(xy 133.35 177.8) (xy 153.67 177.8)
 		)
@@
 	(wire
 		(pts
+			(xy 124.46 193.04) (xy 124.46 196.85)
+		)
+		(stroke
+			(width 0)
+			(type default)
+		)
+	)
+	(wire
+		(pts
 			(xy 115.57 49.53) (xy 121.92 49.53)
 		)
@@
 	(wire
 		(pts
-			(xy 124.46 193.04) (xy 127 193.04)
-		)
-		(stroke
-			(width 0)
-			(type default)
-		)
-	)
-	(wire
-		(pts
 			(xy 90.17 24.13) (xy 96.52 24.13)
 		)
@@
 	(wire
 		(pts
-			(xy 127 190.5) (xy 127 193.04)
-		)
-		(stroke
-			(width 0)
-			(type default)
-		)
-	)
-	(wire
-		(pts
 			(xy 217.17 74.93) (xy 223.52 74.93)
 		)
@@
 	(wire
 		(pts
+			(xy 127 190.5) (xy 127 193.04)
+		)
+		(stroke
+			(width 0)
+			(type default)
+		)
+	)
+	(wire
+		(pts
 			(xy 124.46 170.18) (xy 146.05 170.18)
 		)
@@
 	)
 	(symbol
-		(lib_id "power:GND")
-		(at 127 195.58 0)
-		(unit 1)
-		(exclude_from_sim no)
-		(in_bom yes)
-		(on_board yes)
-		(dnp no)
-		(fields_autoplaced yes)
-		(property "Reference" "#PWR034"
-			(at 127 201.93 0)
-			(effects
-				(font
-					(size 1.27 1.27)
-				)
-				(hide yes)
-			)
-		)
-		(property "Value" "GND"
-			(at 127 200.66 0)
-			(effects
-				(font
-					(size 1.27 1.27)
-				)
-			)
-		)
-		(property "Footprint" ""
-			(at 127 195.58 0)
-			(effects
-				(font
-					(size 1.27 1.27)
-				)
-				(hide yes)
-			)
-		)
-		(property "Datasheet" ""
-			(at 127 195.58 0)
-			(effects
-				(font
-					(size 1.27 1.27)
-				)
-				(hide yes)
-			)
-		)
-		(property "Description" "Power symbol creates a global label with name \"GND\" , ground"
-			(at 127 195.58 0)
-			(effects
-				(font
-					(size 1.27 1.27)
-				)
-				(hide yes)
-			)
-		)
-		(pin "1"
-		)
-		(instances
-			(project "keyboard"
-				(path "/ee756133-ce5d-4302-8df3-762da84ea123"
-					(reference "#PWR034")
-					(unit 1)
-				)
-			)
-		)
-	)
-	(symbol
 		(lib_id "MX_Alps_Hybrid:MX-NoLED")
 		(at 111.76 127 0)
@@
 					(unit 1)
 				)
+			)
+		)
+	)
+	(symbol
+		(lib_id "power:Earth")
+		(at 124.46 196.85 0)
+		(unit 1)
+		(exclude_from_sim no)
+		(in_bom yes)
+		(on_board yes)
+		(dnp no)
+		(fields_autoplaced yes)
+		(property "Reference" "#PWR01"
+			(at 124.46 203.2 0)
+			(effects
+				(font
+					(size 1.27 1.27)
+				)
+				(hide yes)
+			)
+		)
+		(property "Value" "Earth"
+			(at 124.46 201.93 0)
+			(effects
+				(font
+					(size 1.27 1.27)
+				)
+			)
+		)
+		(property "Footprint" ""
+			(at 124.46 196.85 0)
+			(effects
+				(font
+					(size 1.27 1.27)
+				)
+				(hide yes)
+			)
+		)
+		(property "Datasheet" "~"
+			(at 124.46 196.85 0)
+			(effects
+				(font
+					(size 1.27 1.27)
+				)
+				(hide yes)
+			)
+		)
+		(property "Description" "Power symbol creates a global label with name \"Earth\""
+			(at 124.46 196.85 0)
+			(effects
+				(font
+					(size 1.27 1.27)
+				)
+				(hide yes)
+			)
+		)
+		(pin "1"
+		)
+		(instances
+			(project ""
+				(path "/ee756133-ce5d-4302-8df3-762da84ea123"
+					(reference "#PWR01")
+					(unit 1)
+				)

Commit message: Update.
Connections:
- net GND: now also R10.2, R9.2, USB2.1 (GND), USB2.12 (GND)
Changed lines of the file:
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@@
 	)
 	(junction
+		(at 142.24 193.04)
+		(diameter 0)
+		(color 0 0 0 0)
+	)
+	(junction
 		(at 160.02 218.44)
 		(diameter 0)
@@
 	(wire
 		(pts
-			(xy 137.16 193.04) (xy 146.05 193.04)
+			(xy 137.16 193.04) (xy 142.24 193.04)
 		)
 		(stroke
@@
 	(wire
 		(pts
+			(xy 142.24 193.04) (xy 146.05 193.04)
+		)
+		(stroke
+			(width 0)
+			(type default)
+		)
+	)
+	(wire
+		(pts
 			(xy 147.32 100.33) (xy 147.32 74.93)
 		)
@@
 					(unit 1)
 				)
+			)
+		)
+	)
+	(symbol
+		(lib_id "power:GND")
+		(at 142.24 193.04 0)
+		(unit 1)
+		(exclude_from_sim no)
+		(in_bom yes)
+		(on_board yes)
+		(dnp no)
+		(fields_autoplaced yes)
+		(property "Reference" "#PWR02"
+			(at 142.24 199.39 0)
+			(effects
+				(font
+					(size 1.27 1.27)
+				)
+				(hide yes)
+			)
+		)
+		(property "Value" "GND"
+			(at 142.24 198.12 0)
+			(effects
+				(font
+					(size 1.27 1.27)
+				)
+			)
+		)
+		(property "Footprint" ""
+			(at 142.24 193.04 0)
+			(effects
+				(font
+					(size 1.27 1.27)
+				)
+				(hide yes)
+			)
+		)
+		(property "Datasheet" ""
+			(at 142.24 193.04 0)
+			(effects
+				(font
+					(size 1.27 1.27)
+				)
+				(hide yes)
+			)
+		)
+		(property "Description" "Power symbol creates a global label with name \"GND\" , ground"
+			(at 142.24 193.04 0)
+			(effects
+				(font
+					(size 1.27 1.27)
+				)
+				(hide yes)
+			)
+		)
+		(pin "1"
+		)
+		(instances
+			(project ""
+				(path "/ee756133-ce5d-4302-8df3-762da84ea123"
+					(reference "#PWR02")
+					(unit 1)
+				)

Commit message: Update annotations.
Parts:
- D_1: renamed from D_0; JLCPCB Part (none) -> C2128
- D_10: renamed from D_9; JLCPCB Part (none) -> C2128
- D_11: renamed from D_10; JLCPCB Part (none) -> C2128
- D_12: renamed from D_11; JLCPCB Part (none) -> C2128
- D_13: renamed from D_12; JLCPCB Part (none) -> C2128
- D_14: renamed from D_13; JLCPCB Part (none) -> C2128
- D_15: renamed from D_14; JLCPCB Part (none) -> C2128
- D_16: renamed from D_15; JLCPCB Part (none) -> C2128
- D_17: renamed from D_16; JLCPCB Part (none) -> C2128
- D_18: renamed from D_17; JLCPCB Part (none) -> C2128
- D_19: renamed from D_18; JLCPCB Part (none) -> C2128
- D_2: renamed from D_1; JLCPCB Part (none) -> C2128
- D_20: renamed from D_19; JLCPCB Part (none) -> C2128
- D_21: renamed from D_20; JLCPCB Part (none) -> C2128
- D_22: renamed from D_21; JLCPCB Part (none) -> C2128
- D_23: renamed from D_22; JLCPCB Part (none) -> C2128
- D_24: renamed from D_23; JLCPCB Part (none) -> C2128
- D_25: renamed from D_24; JLCPCB Part (none) -> C2128
- D_26: renamed from D_25; JLCPCB Part (none) -> C2128
- D_27: renamed from D_26; JLCPCB Part (none) -> C2128
- D_28: renamed from D_27; JLCPCB Part (none) -> C2128
- D_29: renamed from D_28; JLCPCB Part (none) -> C2128
- D_3: renamed from D_2; JLCPCB Part (none) -> C2128
- D_30: renamed from D_29; JLCPCB Part (none) -> C2128
- D_31: renamed from D_30; JLCPCB Part (none) -> C2128
- D_32: renamed from D_31; JLCPCB Part (none) -> C2128
- D_33: renamed from D_32; JLCPCB Part (none) -> C2128
- D_34: renamed from D_33; JLCPCB Part (none) -> C2128
- D_35: renamed from D_34; JLCPCB Part (none) -> C2128
- D_36: renamed from D_35; JLCPCB Part (none) -> C2128
- D_37: renamed from D_36; JLCPCB Part (none) -> C2128
- D_38: renamed from D_37; JLCPCB Part (none) -> C2128
- D_39: renamed from D_38; JLCPCB Part (none) -> C2128
- D_4: renamed from D_3; JLCPCB Part (none) -> C2128
- D_40: renamed from D_39; JLCPCB Part (none) -> C2128
- D_41: renamed from D_40; JLCPCB Part (none) -> C2128
- D_42: renamed from D_41; JLCPCB Part (none) -> C2128
- D_43: renamed from D_42; JLCPCB Part (none) -> C2128
- D_44: renamed from D_43; JLCPCB Part (none) -> C2128
- D_45: renamed from D_44; JLCPCB Part (none) -> C2128
- D_46: renamed from D_45; JLCPCB Part (none) -> C2128
- D_47: renamed from D_46; JLCPCB Part (none) -> C2128
- D_48: renamed from D_47; JLCPCB Part (none) -> C2128
- D_49: renamed from D_48; JLCPCB Part (none) -> C2128
- D_5: renamed from D_4; JLCPCB Part (none) -> C2128
- D_50: renamed from D_49; JLCPCB Part (none) -> C2128
- D_51: renamed from D_50; JLCPCB Part (none) -> C2128
- D_52: renamed from D_51; JLCPCB Part (none) -> C2128
- D_53: renamed from D_52; JLCPCB Part (none) -> C2128
- D_54: renamed from D_53; JLCPCB Part (none) -> C2128
- D_55: renamed from D_54; JLCPCB Part (none) -> C2128
- D_56: renamed from D_55; JLCPCB Part (none) -> C2128
- D_57: renamed from D_56; JLCPCB Part (none) -> C2128
- D_58: renamed from D_57; JLCPCB Part (none) -> C2128
- D_59: renamed from D_58; JLCPCB Part (none) -> C2128
- D_6: renamed from D_5; JLCPCB Part (none) -> C2128
- D_60: renamed from D_59; JLCPCB Part (none) -> C2128
- D_61: renamed from D_60; JLCPCB Part (none) -> C2128
- D_62: renamed from D_61; JLCPCB Part (none) -> C2128
- D_7: renamed from D_6; JLCPCB Part (none) -> C2128
- D_8: renamed from D_7; JLCPCB Part (none) -> C2128
- D_9: renamed from D_8; JLCPCB Part (none) -> C2128
- J1: renamed from J2; footprint random-keyboard-parts:Reset_Pretty-Mask -> local:Reset_Pretty-Mask_rp2040
- K_1: renamed from K_0; value KEYSW -> esc; footprint PCM_Switch_Keyboard_Hotswap_Kailh:SW_Hotswap_Kailh_Choc_V1V2 -> local:SW_Hotswap_Kailh_Choc_V1V2_annotated
- K_10: renamed from K_9; value KEYSW -> 9; footprint PCM_Switch_Keyboard_Hotswap_Kailh:SW_Hotswap_Kailh_Choc_V1V2 -> local:SW_Hotswap_Kailh_Choc_V1V2_annotated
- K_11: renamed from K_10; value KEYSW -> 0; footprint PCM_Switch_Keyboard_Hotswap_Kailh:SW_Hotswap_Kailh_Choc_V1V2 -> local:SW_Hotswap_Kailh_Choc_V1V2_annotated
- K_12: renamed from K_11; value KEYSW -> minus; footprint PCM_Switch_Keyboard_Hotswap_Kailh:SW_Hotswap_Kailh_Choc_V1V2 -> local:SW_Hotswap_Kailh_Choc_V1V2_annotated
- K_13: renamed from K_12; value KEYSW -> equals; footprint PCM_Switch_Keyboard_Hotswap_Kailh:SW_Hotswap_Kailh_Choc_V1V2 -> local:SW_Hotswap_Kailh_Choc_V1V2_annotated
- K_14: renamed from K_13; value KEYSW -> bash; footprint PCM_Switch_Keyboard_Hotswap_Kailh:SW_Hotswap_Kailh_Choc_V1V2 -> local:SW_Hotswap_Kailh_Choc_V1V2_annotated
- K_15: renamed from K_14; value KEYSW -> grave; footprint PCM_Switch_Keyboard_Hotswap_Kailh:SW_Hotswap_Kailh_Choc_V1V2 -> local:SW_Hotswap_Kailh_Choc_V1V2_annotated
- K_16: renamed from K_15; value KEYSW -> tab; footprint PCM_Switch_Keyboard_Hotswap_Kailh:SW_Hotswap_Kailh_Choc_V1V2 -> local:SW_Hotswap_Kailh_Choc_V1V2_annotated
- K_17: renamed from K_16; value KEYSW -> q; footprint PCM_Switch_Keyboard_Hotswap_Kailh:SW_Hotswap_Kailh_Choc_V1V2 -> local:SW_Hotswap_Kailh_Choc_V1V2_annotated
- K_18: renamed from K_17; value KEYSW -> w; footprint PCM_Switch_Keyboard_Hotswap_Kailh:SW_Hotswap_Kailh_Choc_V1V2 -> local:SW_Hotswap_Kailh_Choc_V1V2_annotated
- K_19: renamed from K_18; value KEYSW -> e; footprint PCM_Switch_Keyboard_Hotswap_Kailh:SW_Hotswap_Kailh_Choc_V1V2 -> local:SW_Hotswap_Kailh_Choc_V1V2_annotated
- K_2: renamed from K_1; value KEYSW -> 1; footprint PCM_Switch_Keyboard_Hotswap_Kailh:SW_Hotswap_Kailh_Choc_V1V2 -> local:SW_Hotswap_Kailh_Choc_V1V2_annotated
- K_20: renamed from K_19; value KEYSW -> r; footprint PCM_Switch_Keyboard_Hotswap_Kailh:SW_Hotswap_Kailh_Choc_V1V2 -> local:SW_Hotswap_Kailh_Choc_V1V2_annotated
- K_21: renamed from K_20; value KEYSW -> t; footprint PCM_Switch_Keyboard_Hotswap_Kailh:SW_Hotswap_Kailh_Choc_V1V2 -> local:SW_Hotswap_Kailh_Choc_V1V2_annotated
- K_22: renamed from K_21; value KEYSW -> y; footprint PCM_Switch_Keyboard_Hotswap_Kailh:SW_Hotswap_Kailh_Choc_V1V2 -> local:SW_Hotswap_Kailh_Choc_V1V2_annotated
- K_23: renamed from K_22; value KEYSW -> u; footprint PCM_Switch_Keyboard_Hotswap_Kailh:SW_Hotswap_Kailh_Choc_V1V2 -> local:SW_Hotswap_Kailh_Choc_V1V2_annotated
- K_24: renamed from K_23; value KEYSW -> i; footprint PCM_Switch_Keyboard_Hotswap_Kailh:SW_Hotswap_Kailh_Choc_V1V2 -> local:SW_Hotswap_Kailh_Choc_V1V2_annotated
- K_25: renamed from K_24; value KEYSW -> o; footprint PCM_Switch_Keyboard_Hotswap_Kailh:SW_Hotswap_Kailh_Choc_V1V2 -> local:SW_Hotswap_Kailh_Choc_V1V2_annotated
- K_26: renamed from K_25; value KEYSW -> p; footprint PCM_Switch_Keyboard_Hotswap_Kailh:SW_Hotswap_Kailh_Choc_V1V2 -> local:SW_Hotswap_Kailh_Choc_V1V2_annotated
- K_27: renamed from K_26; value KEYSW -> l_brace; footprint PCM_Switch_Keyboard_Hotswap_Kailh:SW_Hotswap_Kailh_Choc_V1V2 -> local:SW_Hotswap_Kailh_Choc_V1V2_annotated
- K_28: renamed from K_27; value KEYSW -> r_brace; footprint PCM_Switch_Keyboard_Hotswap_Kailh:SW_Hotswap_Kailh_Choc_V1V2 -> local:SW_Hotswap_Kailh_Choc_V1V2_annotated
- K_29: renamed from K_28; value KEYSW -> bksp; footprint PCM_Switch_Keyboard_Hotswap_Kailh:SW_Hotswap_Kailh_Choc_V1V2 -> local:SW_Hotswap_Kailh_Choc_V1V2_annotated
- K_3: renamed from K_2; value KEYSW -> 2; footprint PCM_Switch_Keyboard_Hotswap_Kailh:SW_Hotswap_Kailh_Choc_V1V2 -> local:SW_Hotswap_Kailh_Choc_V1V2_annotated
- K_30: renamed from K_29; value KEYSW -> l_ctrl; footprint PCM_Switch_Keyboard_Hotswap_Kailh:SW_Hotswap_Kailh_Choc_V1V2 -> local:SW_Hotswap_Kailh_Choc_V1V2_annotated
- K_31: renamed from K_30; value KEYSW -> a; footprint PCM_Switch_Keyboard_Hotswap_Kailh:SW_Hotswap_Kailh_Choc_V1V2 -> local:SW_Hotswap_Kailh_Choc_V1V2_annotated
- K_32: renamed from K_31; value KEYSW -> s; footprint PCM_Switch_Keyboard_Hotswap_Kailh:SW_Hotswap_Kailh_Choc_V1V2 -> local:SW_Hotswap_Kailh_Choc_V1V2_annotated
- K_33: renamed from K_32; value KEYSW -> d; footprint PCM_Switch_Keyboard_Hotswap_Kailh:SW_Hotswap_Kailh_Choc_V1V2 -> local:SW_Hotswap_Kailh_Choc_V1V2_annotated
- K_34: renamed from K_33; value KEYSW -> f; footprint PCM_Switch_Keyboard_Hotswap_Kailh:SW_Hotswap_Kailh_Choc_V1V2 -> local:SW_Hotswap_Kailh_Choc_V1V2_annotated
- K_35: renamed from K_34; value KEYSW -> g; footprint PCM_Switch_Keyboard_Hotswap_Kailh:SW_Hotswap_Kailh_Choc_V1V2 -> local:SW_Hotswap_Kailh_Choc_V1V2_annotated
- K_36: renamed from K_35; value KEYSW -> h; footprint PCM_Switch_Keyboard_Hotswap_Kailh:SW_Hotswap_Kailh_Choc_V1V2 -> local:SW_Hotswap_Kailh_Choc_V1V2_annotated
- K_37: renamed from K_36; value KEYSW -> j; footprint PCM_Switch_Keyboard_Hotswap_Kailh:SW_Hotswap_Kailh_Choc_V1V2 -> local:SW_Hotswap_Kailh_Choc_V1V2_annotated
- K_38: renamed from K_37; value KEYSW -> k; footprint PCM_Switch_Keyboard_Hotswap_Kailh:SW_Hotswap_Kailh_Choc_V1V2 -> local:SW_Hotswap_Kailh_Choc_V1V2_annotated
- K_39: renamed from K_38; value KEYSW -> l; footprint PCM_Switch_Keyboard_Hotswap_Kailh:SW_Hotswap_Kailh_Choc_V1V2 -> local:SW_Hotswap_Kailh_Choc_V1V2_annotated
- K_4: renamed from K_3; value KEYSW -> 3; footprint PCM_Switch_Keyboard_Hotswap_Kailh:SW_Hotswap_Kailh_Choc_V1V2 -> local:SW_Hotswap_Kailh_Choc_V1V2_annotated
- K_40: renamed from K_39; value KEYSW -> semi; footprint PCM_Switch_Keyboard_Hotswap_Kailh:SW_Hotswap_Kailh_Choc_V1V2 -> local:SW_Hotswap_Kailh_Choc_V1V2_annotated
- K_41: renamed from K_40; value KEYSW -> quote; footprint PCM_Switch_Keyboard_Hotswap_Kailh:SW_Hotswap_Kailh_Choc_V1V2 -> local:SW_Hotswap_Kailh_Choc_V1V2_annotated
- K_42: renamed from K_41; value KEYSW -> enter; footprint PCM_Switch_Keyboard_Hotswap_Kailh:SW_Hotswap_Kailh_Choc_V1V2 -> local:SW_Hotswap_Kailh_Choc_V1V2_annotated
- K_43: renamed from K_42; value KEYSW -> l_shift; footprint PCM_Switch_Keyboard_Hotswap_Kailh:SW_Hotswap_Kailh_Choc_V1V2 -> local:SW_Hotswap_Kailh_Choc_V1V2_annotated
- K_44: renamed from K_43; value KEYSW -> z; footprint PCM_Switch_Keyboard_Hotswap_Kailh:SW_Hotswap_Kailh_Choc_V1V2 -> local:SW_Hotswap_Kailh_Choc_V1V2_annotated
- K_45: renamed from K_44; value KEYSW -> x; footprint PCM_Switch_Keyboard_Hotswap_Kailh:SW_Hotswap_Kailh_Choc_V1V2 -> local:SW_Hotswap_Kailh_Choc_V1V2_annotated
- K_46: renamed from K_45; value KEYSW -> c; footprint PCM_Switch_Keyboard_Hotswap_Kailh:SW_Hotswap_Kailh_Choc_V1V2 -> local:SW_Hotswap_Kailh_Choc_V1V2_annotated
- K_47: renamed from K_46; value KEYSW -> v; footprint PCM_Switch_Keyboard_Hotswap_Kailh:SW_Hotswap_Kailh_Choc_V1V2 -> local:SW_Hotswap_Kailh_Choc_V1V2_annotated
- K_48: renamed from K_47; value KEYSW -> b; footprint PCM_Switch_Keyboard_Hotswap_Kailh:SW_Hotswap_Kailh_Choc_V1V2 -> local:SW_Hotswap_Kailh_Choc_V1V2_annotated
- K_49: renamed from K_48; value KEYSW -> n; footprint PCM_Switch_Keyboard_Hotswap_Kailh:SW_Hotswap_Kailh_Choc_V1V2 -> local:SW_Hotswap_Kailh_Choc_V1V2_annotated
- K_5: renamed from K_4; value KEYSW -> 4; footprint PCM_Switch_Keyboard_Hotswap_Kailh:SW_Hotswap_Kailh_Choc_V1V2 -> local:SW_Hotswap_Kailh_Choc_V1V2_annotated
- K_50: renamed from K_49; value KEYSW -> m; footprint PCM_Switch_Keyboard_Hotswap_Kailh:SW_Hotswap_Kailh_Choc_V1V2 -> local:SW_Hotswap_Kailh_Choc_V1V2_annotated
- K_51: renamed from K_50; value KEYSW -> comma; footprint PCM_Switch_Keyboard_Hotswap_Kailh:SW_Hotswap_Kailh_Choc_V1V2 -> local:SW_Hotswap_Kailh_Choc_V1V2_annotated
- K_52: renamed from K_51; value KEYSW -> dot; footprint PCM_Switch_Keyboard_Hotswap_Kailh:SW_Hotswap_Kailh_Choc_V1V2 -> local:SW_Hotswap_Kailh_Choc_V1V2_annotated
- K_53: renamed from K_52; value KEYSW -> slash; footprint PCM_Switch_Keyboard_Hotswap_Kailh:SW_Hotswap_Kailh_Choc_V1V2 -> local:SW_Hotswap_Kailh_Choc_V1V2_annotated
- K_54: renamed from K_53; value KEYSW -> r_shift; footprint PCM_Switch_Keyboard_Hotswap_Kailh:SW_Hotswap_Kailh_Choc_V1V2 -> local:SW_Hotswap_Kailh_Choc_V1V2_annotated
- K_55: renamed from K_54; value KEYSW -> mo1; footprint PCM_Switch_Keyboard_Hotswap_Kailh:SW_Hotswap_Kailh_Choc_V1V2 -> local:SW_Hotswap_Kailh_Choc_V1V2_annotated
- K_56: renamed from K_55; value KEYSW -> l_gui; footprint PCM_Switch_Keyboard_Hotswap_Kailh:SW_Hotswap_Kailh_Choc_V1V2 -> local:SW_Hotswap_Kailh_Choc_V1V2_annotated
- K_57: renamed from K_56; value KEYSW -> l_alt; footprint PCM_Switch_Keyboard_Hotswap_Kailh:SW_Hotswap_Kailh_Choc_V1V2 -> local:SW_Hotswap_Kailh_Choc_V1V2_annotated
- K_58: renamed from K_57; value KEYSW -> space; footprint PCM_Switch_Keyboard_Hotswap_Kailh:SW_Hotswap_Kailh_Choc_V1V2 -> local:SW_Hotswap_Kailh_Choc_V1V2_annotated
- K_59: renamed from K_58; value KEYSW -> mo2; footprint PCM_Switch_Keyboard_Hotswap_Kailh:SW_Hotswap_Kailh_Choc_V1V2 -> local:SW_Hotswap_Kailh_Choc_V1V2_annotated
- K_6: renamed from K_5; value KEYSW -> 5; footprint PCM_Switch_Keyboard_Hotswap_Kailh:SW_Hotswap_Kailh_Choc_V1V2 -> local:SW_Hotswap_Kailh_Choc_V1V2_annotated
- K_60: renamed from K_59; value KEYSW -> space; footprint PCM_Switch_Keyboard_Hotswap_Kailh:SW_Hotswap_Kailh_Choc_V1V2 -> local:SW_Hotswap_Kailh_Choc_V1V2_annotated
- K_61: renamed from K_60; value KEYSW -> r_alt; footprint PCM_Switch_Keyboard_Hotswap_Kailh:SW_Hotswap_Kailh_Choc_V1V2 -> local:SW_Hotswap_Kailh_Choc_V1V2_annotated
- K_62: renamed from K_61; value KEYSW -> r_ctrl; footprint PCM_Switch_Keyboard_Hotswap_Kailh:SW_Hotswap_Kailh_Choc_V1V2 -> local:SW_Hotswap_Kailh_Choc_V1V2_annotated
- K_7: renamed from K_6; value KEYSW -> 6; footprint PCM_Switch_Keyboard_Hotswap_Kailh:SW_Hotswap_Kailh_Choc_V1V2 -> local:SW_Hotswap_Kailh_Choc_V1V2_annotated
- K_8: renamed from K_7; value KEYSW -> 7; footprint PCM_Switch_Keyboard_Hotswap_Kailh:SW_Hotswap_Kailh_Choc_V1V2 -> local:SW_Hotswap_Kailh_Choc_V1V2_annotated
- K_9: renamed from K_8; value KEYSW -> 8; footprint PCM_Switch_Keyboard_Hotswap_Kailh:SW_Hotswap_Kailh_Choc_V1V2 -> local:SW_Hotswap_Kailh_Choc_V1V2_annotated
- USB1: renamed from USB2; JLCPCB Part (none) -> C165948
- renumbered C30 to C1, C22 to C10, C24 to C11, C25 to C12, C27 to C13, C28 to C14, C29 to C15, C32 to C16, C23 to C2, C26 to C3, C31 to C4, C17 to C5, C18 to C6, C19 to C7, C20 to C8, C21 to C9, F2 to F1, FB2 to FB1, R8 to R1, R14 to R2, R11 to R3, R12 to R4, R9 to R5, R10 to R6, R13 to R7, SW2 to SW1, U7 to U1, U6 to U2, U5 to U3, U8 to U4, Y2 to Y1
Connections:
- net GPIO22: now also U3.34 (GPIO22)
- net GPIO8: now reaches U3.11 (GPIO8)
- net GPIO9: now reaches U3.12 (GPIO9)
- net GPIO10: now reaches U3.13 (GPIO10)
- net GPIO11: now reaches U3.14 (GPIO11)
- net GPIO12: now reaches U3.15 (GPIO12)
