File: boethia60/boethia60.kicad_sch (KiCad schematic)
At the start: 157 parts, among them J1 Conn_01x06, SW1 SW_Push, U1 NCP1117-3.3_SOT223, U2 PRTR5V0U2X, U3 RP2040, U4 W25Q128JVS, Y1 Crystal_GND24_Small

Commit message: Fix incorrect package BOM item.
Parts:
- C10, C11, C12, C14, C15, C16, C6, C7, C8, C9: JLCPCB Part C14663 -> C1525
Changed lines of the file:
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@@
 			)
 		)
-		(property "JLCPCB Part" "C14663"
+		(property "JLCPCB Part" "C1525"
 			(at 186.69 214.63 0)
 			(effects
@@
 			)
 		)
-		(property "JLCPCB Part" "C14663"
+		(property "JLCPCB Part" "C1525"
 			(at 199.39 214.63 0)
 			(effects
@@
 			)
 		)
-		(property "JLCPCB Part" "C14663"
+		(property "JLCPCB Part" "C1525"
 			(at 134.62 214.63 0)
 			(effects
@@
 			)
 		)
-		(property "JLCPCB Part" "C14663"
+		(property "JLCPCB Part" "C1525"
 			(at 238.76 214.63 0)
 			(effects
@@
 			)
 		)
-		(property "JLCPCB Part" "C14663"
+		(property "JLCPCB Part" "C1525"
 			(at 226.06 214.63 0)
 			(effects
@@
 			)
 		)
-		(property "JLCPCB Part" "C14663"
+		(property "JLCPCB Part" "C1525"
 			(at 160.02 214.63 0)
 			(effects
@@
 			)
 		)
-		(property "JLCPCB Part" "C14663"
+		(property "JLCPCB Part" "C1525"
 			(at 121.92 214.63 0)
 			(effects
@@
 			)
 		)
-		(property "JLCPCB Part" "C14663"
+		(property "JLCPCB Part" "C1525"
 			(at 173.99 214.63 0)
 			(effects
@@
 			)
 		)
-		(property "JLCPCB Part" "C14663"
+		(property "JLCPCB Part" "C1525"
 			(at 147.32 214.63 0)
 			(effects
@@
 			)
 		)
-		(property "JLCPCB Part" "C14663"
+		(property "JLCPCB Part" "C1525"
 			(at 270.51 256.54 0)
 			(effects
